File: Project Architecture.kicad_sch (KiCad schematic)
At the start: 67 parts, among them J401 EBWA-02-B, J701 PS0519, J702 EBWA-02-B, Q101 BC549, Q401 Si4944DY, SW501 SW_HELP, U201 LM393, U601 Photon 2, U701 L7805

Commit message: feat: release
Other:
- moved on the sheet: TP101, TP201
Changed lines of the file:
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@@
 	)
 	(junction
-		(at 145.415 63.5)
-		(diameter 0)
-		(color 0 0 0 0)
-	)
-	(junction
 		(at 154.94 119.38)
 		(diameter 0)
@@
 	)
 	(junction
+		(at 146.05 63.5)
+		(diameter 0)
+		(color 0 0 0 0)
+	)
+	(junction
 		(at 312.42 127)
 		(diameter 0)
@@
 	(wire
 		(pts
-			(xy 251.46 55.245) (xy 251.46 63.5)
+			(xy 251.46 54.61) (xy 251.46 63.5)
 		)
 		(stroke
@@
 	(wire
 		(pts
+			(xy 146.05 63.5) (xy 147.32 63.5)
+		)
+		(stroke
+			(width 0)
+			(type default)
+		)
+	)
+	(wire
+		(pts
 			(xy 257.81 124.46) (xy 260.35 124.46)
 		)
@@
 	(wire
 		(pts
-			(xy 145.415 63.5) (xy 147.32 63.5)
-		)
-		(stroke
-			(width 0)
-			(type default)
-		)
-	)
-	(wire
-		(pts
 			(xy 88.9 69.85) (xy 97.79 69.85)
 		)
@@
 	(wire
 		(pts
-			(xy 135.89 63.5) (xy 145.415 63.5)
+			(xy 135.89 63.5) (xy 146.05 63.5)
 		)
 		(stroke
@@
 	(wire
 		(pts
-			(xy 145.415 55.245) (xy 145.415 63.5)
+			(xy 146.05 54.61) (xy 146.05 63.5)
 		)
 		(stroke
@@
 	(symbol
 		(lib_id "Connector:TestPoint")
-		(at 145.415 55.245 0)
+		(at 146.05 54.61 0)
 		(unit 1)
 		(exclude_from_sim no)
@@
 		(fields_autoplaced yes)
 		(property "Reference" "TP101"
-			(at 147.32 50.6729 0)
+			(at 147.955 50.0379 0)
 			(effects
 				(font
@@
 		)
 		(property "Value" "AMP_OUT"
-			(at 147.32 53.2129 0)
+			(at 147.955 52.5779 0)
 			(effects
 				(font
@@
 		)
 		(property "Footprint" "RD-Testpoints:TestPoint_Loop_D1.80mm_Drill1.0mm_Beaded"
-			(at 150.495 55.245 0)
+			(at 151.13 54.61 0)
 			(effects
 				(font
@@
 		)
 		(property "Datasheet" "~"
-			(at 150.495 55.245 0)
+			(at 151.13 54.61 0)
 			(effects
 				(font
@@
 		)
 		(property "Description" "test point"
-			(at 145.415 55.245 0)
+			(at 146.05 54.61 0)
 			(effects
 				(font
@@
 	(symbol
 		(lib_id "Connector:TestPoint")
-		(at 251.46 55.245 0)
+		(at 251.46 54.61 0)
 		(unit 1)
 		(exclude_from_sim no)
@@
 		(fields_autoplaced yes)
 		(property "Reference" "TP201"
-			(at 253.365 50.6729 0)
+			(at 253.365 50.0379 0)
 			(effects
 				(font
@@
 		)
 		(property "Value" "ENV"
-			(at 253.365 53.2129 0)
+			(at 253.365 52.5779 0)
 			(effects
 				(font
@@
 		)
 		(property "Footprint" "RD-Testpoints:TestPoint_Loop_D1.80mm_Drill1.0mm_Beaded"
-			(at 256.54 55.245 0)
+			(at 256.54 54.61 0)
 			(effects
 				(font
@@
 		)
 		(property "Datasheet" "~"
-			(at 256.54 55.245 0)
+			(at 256.54 54.61 0)
 			(effects
 				(font
@@
 		)
 		(property "Description" "test point"
-			(at 251.46 55.245 0)
+			(at 251.46 54.61 0)
 			(effects
 				(font

Commit message: fix: change status led wiring and improve 12V input protection
Parts:
- added HS701: Heatsink, RD-Heatsinks:Heatsink_6073B_19x9.5mm, symbol Mechanical:Heatsink
- D701: value P4KE16AC -> P4KE16; footprint Diode_THT:D_DO-41_SOD81_P7.62mm_Horizontal -> Diode_THT:D_DO-41_SOD81_P10.16mm_Horizontal; symbol Device:D_TVS -> Device:D_Zener
- F701: value 1A M205 -> 500mA M205
- ID901: footprint RD-Symbols-Silkscreen:STACKUP_ID_2L_SML -> RD-Symbols-Silkscreen:STACKUP_ID_2L
Connections:
- net +12V_FUSED: now also D701.1 (K)
- net +12V_IN: no longer D701.1 (A1)
- net LED_GRN: now also U601.20 (D3); no longer U601.15 (TX)
- net LED_RED: now also U601.21 (D4); no longer U601.14 (RX)
Other:
- moved on the sheet: D701, F701
Changed lines of the file:
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@@
 	)
 	(junction
-		(at 227.33 185.42)
-		(diameter 0)
-		(color 0 0 0 0)
-	)
-	(junction
 		(at 137.16 195.58)
 		(diameter 0)
@@
 	)
 	(junction
+		(at 237.49 185.42)
+		(diameter 0)
+		(color 0 0 0 0)
+	)
+	(junction
 		(at 251.46 63.5)
 		(diameter 0)
@@
 	)
 	(no_connect
+		(at 82.55 215.9)
+	)
+	(no_connect
 		(at 107.95 198.12)
 	)
@@
 	)
 	(no_connect
+		(at 82.55 213.36)
+	)
+	(no_connect
 		(at 107.95 215.9)
 	)
@@
 	)
 	(no_connect
-		(at 107.95 208.28)
-	)
-	(no_connect
 		(at 82.55 185.42)
 	)
@@
 		(at 82.55 180.34)
 	)
-	(no_connect
-		(at 107.95 210.82)
-	)
 	(wire
 		(pts
@@
 	(wire
 		(pts
-			(xy 237.49 185.42) (xy 240.03 185.42)
+			(xy 234.95 185.42) (xy 237.49 185.42)
 		)
 		(stroke
@@
 	(wire
 		(pts
+			(xy 237.49 185.42) (xy 237.49 191.77)
+		)
+		(stroke
+			(width 0)
+			(type default)
+		)
+	)
+	(wire
+		(pts
 			(xy 158.75 63.5) (xy 158.75 66.04)
 		)
@@
 	(wire
 		(pts
-			(xy 217.17 66.04) (xy 217.17 68.58)
+			(xy 237.49 185.42) (xy 240.03 185.42)
 		)
 		(stroke
@@
 	(wire
 		(pts
-			(xy 69.85 213.36) (xy 82.55 213.36)
+			(xy 217.17 66.04) (xy 217.17 68.58)
 		)
 		(stroke
@@
 	(wire
 		(pts
-			(xy 227.33 199.39) (xy 227.33 204.47)
-		)
-		(stroke
-			(width 0)
-			(type default)
-		)
-	)
-	(wire
-		(pts
 			(xy 312.42 73.66) (xy 312.42 78.74)
 		)
@@
 	(wire
 		(pts
-			(xy 227.33 185.42) (xy 229.87 185.42)
-		)
-		(stroke
-			(width 0)
-			(type default)
-		)
-	)
-	(wire
-		(pts
 			(xy 154.94 119.38) (xy 154.94 128.27)
 		)
@@
 	(wire
 		(pts
-			(xy 227.33 185.42) (xy 227.33 191.77)
-		)
-		(stroke
-			(width 0)
-			(type default)
-		)
-	)
-	(wire
-		(pts
 			(xy 254 185.42) (xy 254 191.77)
 		)
@@
 	(wire
 		(pts
+			(xy 107.95 210.82) (xy 120.65 210.82)
+		)
+		(stroke
+			(width 0)
+			(type default)
+		)
+	)
+	(wire
+		(pts
 			(xy 214.63 137.16) (xy 210.82 137.16)
 		)
@@
 	(wire
 		(pts
-			(xy 147.32 96.52) (xy 147.32 97.79)
+			(xy 237.49 199.39) (xy 237.49 204.47)
 		)
 		(stroke
@@
 	(wire
 		(pts
-			(xy 285.75 185.42) (xy 285.75 194.31)
+			(xy 147.32 96.52) (xy 147.32 97.79)
 		)
 		(stroke
@@
 	(wire
 		(pts
-			(xy 154.94 135.89) (xy 154.94 138.43)
+			(xy 285.75 185.42) (xy 285.75 194.31)
 		)
 		(stroke
@@
 	(wire
 		(pts
-			(xy 222.25 204.47) (xy 227.33 204.47)
+			(xy 154.94 135.89) (xy 154.94 138.43)
 		)
 		(stroke
@@
 	(wire
 		(pts
-			(xy 69.85 215.9) (xy 82.55 215.9)
+			(xy 222.25 204.47) (xy 237.49 204.47)
 		)
 		(stroke
@@
 	(wire
 		(pts
+			(xy 107.95 208.28) (xy 120.65 208.28)
+		)
+		(stroke
+			(width 0)
+			(type default)
+		)
+	)
+	(wire
+		(pts
 			(xy 114.3 69.85) (xy 114.3 72.39)
 		)
@@
 		)
 	)
-	(label "LED_RED"
-		(at 69.85 213.36 0)
+	(label "ADC_NTC"
+		(at 120.65 134.62 180)
 		(effects
 			(font
 				(size 1.27 1.27)
 			)
-			(justify left bottom)
+			(justify right bottom)
 		)
 	)
-	(label "ADC_NTC"
-		(at 120.65 134.62 180)
+	(label "FAN-"
+		(at 210.82 129.54 180)
 		(effects
 			(font
@@
 		)
 	)
-	(label "FAN-"
-		(at 210.82 129.54 180)
+	(label "+12V_FUSED"
+		(at 237.49 191.77 180)
 		(effects
 			(font
@@
 		)
 	)
-	(label "LED_GRN"
-		(at 69.85 215.9 0)
-		(effects
-			(font
-				(size 1.27 1.27)
-			)
-			(justify left bottom)
-		)
-	)
 	(label "ADC_POT"
 		(at 69.85 193.04 0)
@@
 		)
 	)
-	(label "+12V_FUSED"
-		(at 240.03 185.42 90)
+	(label "LED_GRN"
+		(at 120.65 210.82 180)
 		(effects
 			(font
 				(size 1.27 1.27)
 			)
-			(justify left bottom)
+			(justify right bottom)
 		)
 	)
@@
 		)
 	)
+	(label "LED_RED"
+		(at 120.65 208.28 180)
+		(effects
+			(font
+				(size 1.27 1.27)
+			)
+			(justify right bottom)
+		)
+	)
 	(label "PWM_FAN"
 		(at 137.16 139.7 90)
@@
 			)
 		)
-		(property "Footprint" "RD-Symbols-Silkscreen:STACKUP_ID_2L_SML"
+		(property "Footprint" "RD-Symbols-Silkscreen:STACKUP_ID_2L"
 			(at 175.26 194.31 0)
 			(effects
@@
 	(symbol
 		(lib_id "Device:Fuse")
-		(at 233.68 185.42 90)
+		(at 231.14 185.42 90)
 		(unit 1)
 		(exclude_from_sim no)
@@
 		(fields_autoplaced yes)
 		(property "Reference" "F701"
-			(at 233.68 179.07 90)
+			(at 231.14 179.07 90)
 			(effects
 				(font
@@
 			)
 		)
-		(property "Value" "1A M205"
-			(at 233.68 181.61 90)
+		(property "Value" "500mA M205"
+			(at 231.14 181.61 90)
 			(effects
 				(font
@@
 		)
 		(property "Footprint" "Fuse:Fuseholder_Clip-5x20mm_Eaton_1A5601-01_Inline_P20.80x6.76mm_D1.70mm_Horizontal"
-			(at 233.68 187.198 90)
+			(at 231.14 187.198 90)
 			(effects
 				(font
@@
 		)
 		(property "Datasheet" "~"
-			(at 233.68 185.42 0)
+			(at 231.14 185.42 0)
 			(effects
 				(font
@@
 		)
 		(property "Description" "Fuse"
-			(at 233.68 185.42 0)
+			(at 231.14 185.42 0)
 			(effects
 				(font
@@
 	)
 	(symbol
+		(lib_id "Mechanical:Heatsink")
+		(at 298.45 176.53 0)
+		(unit 1)
+		(exclude_from_sim no)
+		(in_bom yes)
+		(on_board yes)
+		(dnp no)
+		(fields_autoplaced yes)
+		(property "Reference" "HS701"
+			(at 302.26 173.3549 0)
+			(effects
+				(font
+					(size 1.27 1.27)
+				)
+				(justify left)
+			)
+		)
+		(property "Value" "Heatsink"
+			(at 302.26 175.8949 0)
+			(effects
+				(font
+					(size 1.27 1.27)
+				)
+				(justify left)
+			)
+		)
+		(property "Footprint" "RD-Heatsinks:Heatsink_6073B_19x9.5mm"
+			(at 298.7548 176.53 0)
+			(effects
+				(font
+					(size 1.27 1.27)
+				)
+				(hide yes)
+			)
+		)
+		(property "Datasheet" "~"
+			(at 298.7548 176.53 0)
+			(effects
+				(font
+					(size 1.27 1.27)
+				)
+				(hide yes)
+			)
+		)
+		(property "Description" "Heatsink"
+			(at 298.45 176.53 0)
+			(effects
+				(font
+					(size 1.27 1.27)
+				)
+				(hide yes)
+			)
+		)
+		(instances
+			(project ""
+				(path "/f9e05184-c88b-4a88-ae9c-ab2bdb32be7c/c5103ceb-5325-4a84-a025-9638a412984e"
+					(reference "HS701")
+					(unit 1)
+				)
+			)
+		)
+	)
+	(symbol
 		(lib_id "Device:C")
 		(at 210.82 66.04 270)
@@
 	)
 	(symbol
-		(lib_id "Device:D_TVS")
-		(at 227.33 195.58 270)
+		(lib_id "Device:D_Zener")
+		(at 237.49 195.58 270)
 		(unit 1)
 		(exclude_from_sim no)
@@
 		(fields_autoplaced yes)
 		(property "Reference" "D701"
-			(at 229.87 194.3099 90)
+			(at 240.03 194.3099 90)
 			(effects
 				(font
@@
 			)
 		)
-		(property "Value" "P4KE16AC"
-			(at 229.87 196.8499 90)
+		(property "Value" "P4KE16"
+			(at 240.03 196.8499 90)
 			(effects
 				(font
@@
 			)
 		)
-		(property "Footprint" "Diode_THT:D_DO-41_SOD81_P7.62mm_Horizontal"
-			(at 227.33 195.58 0)
+		(property "Footprint" "Diode_THT:D_DO-41_SOD81_P10.16mm_Horizontal"
+			(at 237.49 195.58 0)
 			(effects
 				(font
@@
 			)
 		)
-		(property "Datasheet" "https://www.jaycar.com.au/p4ke-13-6v-16a-standoff-400w-ac/p/ZR1162"
-			(at 227.33 195.58 0)
+		(property "Datasheet" "~"
+			(at 237.49 195.58 0)
 			(effects
 				(font
@@
 			)
 		)
-		(property "Description" "Bidirectional transient-voltage-suppression diode"
-			(at 227.33 195.58 0)
+		(property "Description" "DIODE TVS UNIDIRECTIONAL"
+			(at 237.49 195.58 0)
 			(effects
 				(font
@@
 		)
 		(property "Manufacturer" ""
-			(at 227.33 195.58 90)
+			(at 237.49 195.58 90)
 			(effects
 				(font
@@
 		)
 		(property "SPN" ""
-			(at 227.33 195.58 90)
+			(at 237.49 195.58 90)
 			(effects
 				(font
@@
 		)
 		(property "Supplier" ""
-			(at 227.33 195.58 90)
+			(at 237.49 195.58 90)
 			(effects
 				(font
@@
 		)
 		(property "Dielectric" ""
-			(at 227.33 195.58 90)
+			(at 237.49 195.58 90)
 			(effects
 				(font
@@
 		)
 		(instances
-			(project ""
+			(project "Sensor-Node-2-Board"
 				(path "/f9e05184-c88b-4a88-ae9c-ab2bdb32be7c/c5103ceb-5325-4a84-a025-9638a412984e"
 					(reference "D701")
